Commit message: feat(semi_taks_lv1): update motor parameters and add simulation mode
Increase effort limits and velocity limits across all joint types. Update armature values for torso (0.124), shoulder (0.032), and wrist/neck (0.002) motors. Adjust corresponding kp/kv gains and force ranges in MuJoCo XML actuators.

Add simulation-only mode with --sim/--real flags. Extract graphics configuration helper for Linux NVIDIA offload and X11 platform selection. Replace custom viewer with mujoco.viewer.launch_passive

File: configs/robots/semi_taks_lv1/Semi_Taks_LV1.urdf (robot description, URDF)
Before this commit: robot Semi_Taks_LV1, 25 links, 24 joints
Joints:
- joint head_pitch_joint: limit lower=-1.57 upper=1.57 effort=6 velocity=12.57 -> lower=-1.57 upper=1.57 effort=12.5 velocity=47.12388980384689
- joint head_yaw_joint: limit lower=-2.618 upper=2.618 effort=6 velocity=12.57 -> lower=-2.618 upper=2.618 effort=12.5 velocity=47.12388980384689
- joint left_elbow_joint: limit lower=-1.0472 upper=1.5708 effort=30 velocity=3.77 -> lower=-1.0472 upper=1.5708 effort=40 velocity=11.728612573401893
- joint left_shoulder_pitch_joint: limit lower=-3.1415 upper=1.0472 effort=30 velocity=3.77 -> lower=-3.1415 upper=1.0472 effort=40 velocity=11.728612573401893
- joint left_shoulder_roll_joint: limit lower=-1.5882 upper=2.2515 effort=30 velocity=3.77 -> lower=-1.5882 upper=2.2515 effort=40 velocity=11.728612573401893
- joint left_shoulder_yaw_joint: limit lower=-2.618 upper=2.618 effort=30 velocity=3.77 -> lower=-2.618 upper=2.618 effort=40 velocity=11.728612573401893
- joint left_wrist_pitch_joint: limit lower=-1.5708 upper=1.5708 effort=6 velocity=12.57 -> lower=-1.5708 upper=1.5708 effort=12.5 velocity=47.12388980384689
- joint left_wrist_roll_joint: limit lower=-2.67 upper=2.67 effort=6 velocity=12.57 -> lower=-2.67 upper=2.67 effort=12.5 velocity=47.12388980384689
- joint left_wrist_yaw_joint: limit lower=-1.309 upper=1.309 effort=6 velocity=12.57 -> lower=-1.309 upper=1.309 effort=12.5 velocity=47.12388980384689
- joint right_elbow_joint: limit lower=-1.0472 upper=1.5708 effort=30 velocity=3.77 -> lower=-1.0472 upper=1.5708 effort=40 velocity=11.728612573401893
- joint right_shoulder_pitch_joint: limit lower=-3.1415 upper=1.0472 effort=30 velocity=3.77 -> lower=-3.1415 upper=1.0472 effort=40 velocity=11.728612573401893
- joint right_shoulder_roll_joint: limit lower=-2.2515 upper=1.5882 effort=30 velocity=3.77 -> lower=-2.2515 upper=1.5882 effort=40 velocity=11.728612573401893
- joint right_shoulder_yaw_joint: limit lower=-2.618 upper=2.618 effort=30 velocity=3.77 -> lower=-2.618 upper=2.618 effort=40 velocity=11.728612573401893
- joint right_wrist_pitch_joint: limit lower=-1.5708 upper=1.5708 effort=6 velocity=12.57 -> lower=-1.5708 upper=1.5708 effort=12.5 velocity=47.12388980384689
- joint right_wrist_roll_joint: limit lower=-2.67 upper=2.67 effort=6 velocity=12.57 -> lower=-2.67 upper=2.67 effort=12.5 velocity=47.12388980384689
- joint right_wrist_yaw_joint: limit lower=-1.309 upper=1.309 effort=6 velocity=12.57 -> lower=-1.309 upper=1.309 effort=12.5 velocity=47.12388980384689
- joint waist_pitch_joint: limit lower=-0.5236 upper=0.5236 effort=60 velocity=4.19 -> lower=-0.5236 upper=0.5236 effort=97 velocity=12.042771838760872
- joint waist_roll_joint: limit lower=-0.5236 upper=0.5236 effort=60 velocity=4.19 -> lower=-0.5236 upper=0.5236 effort=97 velocity=12.042771838760872
- joint waist_yaw_joint: limit lower=-2.618 upper=2.618 effort=60 velocity=4.19 -> lower=-2.618 upper=2.618 effort=97 velocity=12.042771838760872
